File: eagle/ezlpc-proto.sch (EAGLE design)
At the start: 61 parts, among them J1 MICRO USB, Q1 12Mhz, T1 MMBT3906, U1 PRTR5V0U2X, U2 MIC5225-3.3v, U3 LPC11U35FHI33/501

Commit message: Reduced board height by 0.1" to better fit solderless breadboards.
Connections:
- net AUX-VIN: now also TP29.1; no longer TP30.1
- net GND: now also TP28.1; no longer TP29.1
- net PIO0_10-SWDCLK: now also TP24.1; no longer TP25.1
- net PIO0_21: now also TP1.1; no longer TP2.1
- net PIO0_3-VBUS: now also TP25.1; no longer TP26.1
- net PIO0_5: now also TP26.1; no longer TP28.1
- net PIO0_6-CONNECT: now also TP2.1; no longer TP3.1
- net PIO0_7-LED: now also TP3.1; no longer TP1.1
- net USB-5V: now also TP30.1; no longer TP24.1
Other:
- moved on the sheet: TP1, TP2, TP24, TP25, TP26, TP28, TP29, TP3, TP30
Changed lines of the file:
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@@
 <part name="TP17" library="ezlpc-proto" deviceset="PINHD-1X1" device=""/>
 <part name="TP22" library="ezlpc-proto" deviceset="PINHD-1X1" device=""/>
+<part name="TP25" library="ezlpc-proto" deviceset="PINHD-1X1" device=""/>
+<part name="TP23" library="ezlpc-proto" deviceset="PINHD-1X1" device=""/>
 <part name="TP26" library="ezlpc-proto" deviceset="PINHD-1X1" device=""/>
-<part name="TP23" library="ezlpc-proto" deviceset="PINHD-1X1" device=""/>
-<part name="TP28" library="ezlpc-proto" deviceset="PINHD-1X1" device=""/>
+<part name="TP2" library="ezlpc-proto" deviceset="PINHD-1X1" device=""/>
 <part name="TP3" library="ezlpc-proto" deviceset="PINHD-1X1" device=""/>
-<part name="TP1" library="ezlpc-proto" deviceset="PINHD-1X1" device=""/>
 <part name="TP4" library="ezlpc-proto" deviceset="PINHD-1X1" device=""/>
 <part name="TP5" library="ezlpc-proto" deviceset="PINHD-1X1" device=""/>
-<part name="TP25" library="ezlpc-proto" deviceset="PINHD-1X1" device=""/>
+<part name="TP24" library="ezlpc-proto" deviceset="PINHD-1X1" device=""/>
 <part name="TP7" library="ezlpc-proto" deviceset="PINHD-1X1" device=""/>
 <part name="TP8" library="ezlpc-proto" deviceset="PINHD-1X1" device=""/>
@@
 <part name="TP18" library="ezlpc-proto" deviceset="PINHD-1X1" device=""/>
 <part name="TP21" library="ezlpc-proto" deviceset="PINHD-1X1" device=""/>
-<part name="TP2" library="ezlpc-proto" deviceset="PINHD-1X1" device=""/>
+<part name="TP1" library="ezlpc-proto" deviceset="PINHD-1X1" device=""/>
 <part name="TP6" library="ezlpc-proto" deviceset="PINHD-1X1" device=""/>
 <part name="TP13" library="ezlpc-proto" deviceset="PINHD-1X1" device=""/>
 <part name="TP14" library="ezlpc-proto" deviceset="PINHD-1X1" device=""/>
 <part name="TP19" library="ezlpc-proto" deviceset="PINHD-1X1" device=""/>
-<part name="TP24" library="ezlpc-proto" deviceset="PINHD-1X1" device=""/>
+<part name="TP30" library="ezlpc-proto" deviceset="PINHD-1X1" device=""/>
 <part name="TP27" library="ezlpc-proto" deviceset="PINHD-1X1" device=""/>
-<part name="TP29" library="ezlpc-proto" deviceset="PINHD-1X1" device=""/>
+<part name="TP28" library="ezlpc-proto" deviceset="PINHD-1X1" device=""/>
 <part name="GND16" library="ezlpc-proto" deviceset="GND" device=""/>
 <part name="+3V3" library="ezlpc-proto" deviceset="+3V3" device=""/>
@@
 <part name="U$2" library="ezlpc-proto" deviceset="NC" device=""/>
 <part name="T1" library="ezlpc-proto" deviceset="*-PNP-" device="SOT23-BEC" technology="BC857B" value="MMBT3906"/>
-<part name="TP30" library="ezlpc-proto" deviceset="PINHD-1X1" device=""/>
+<part name="TP29" library="ezlpc-proto" deviceset="PINHD-1X1" device=""/>
 </parts>
 <sheets>
@@
 <instance part="TP17" gate="G$1" x="294.64" y="226.06"/>
 <instance part="TP22" gate="G$1" x="294.64" y="223.52"/>
-<instance part="TP26" gate="G$1" x="294.64" y="220.98"/>
+<instance part="TP25" gate="G$1" x="294.64" y="220.98"/>
 <instance part="TP23" gate="G$1" x="294.64" y="218.44"/>
-<instance part="TP28" gate="G$1" x="294.64" y="215.9"/>
-<instance part="TP3" gate="G$1" x="294.64" y="213.36"/>
-<instance part="TP1" gate="G$1" x="294.64" y="210.82"/>
+<instance part="TP26" gate="G$1" x="294.64" y="215.9"/>
+<instance part="TP2" gate="G$1" x="294.64" y="213.36"/>
+<instance part="TP3" gate="G$1" x="294.64" y="210.82"/>
 <instance part="TP4" gate="G$1" x="294.64" y="205.74"/>
 <instance part="TP5" gate="G$1" x="294.64" y="203.2"/>
-<instance part="TP25" gate="G$1" x="294.64" y="200.66"/>
+<instance part="TP24" gate="G$1" x="294.64" y="200.66"/>
 <instance part="TP7" gate="G$1" x="294.64" y="198.12"/>
 <instance part="TP8" gate="G$1" x="294.64" y="195.58"/>
@@
 <instance part="TP18" gate="G$1" x="294.64" y="175.26"/>
 <instance part="TP21" gate="G$1" x="294.64" y="172.72"/>
-<instance part="TP2" gate="G$1" x="294.64" y="170.18"/>
+<instance part="TP1" gate="G$1" x="294.64" y="170.18"/>
 <instance part="TP6" gate="G$1" x="294.64" y="167.64"/>
 <instance part="TP13" gate="G$1" x="294.64" y="165.1"/>
 <instance part="TP14" gate="G$1" x="294.64" y="157.48"/>
 <instance part="TP19" gate="G$1" x="294.64" y="154.94"/>
-<instance part="TP24" gate="G$1" x="294.64" y="142.24"/>
+<instance part="TP30" gate="G$1" x="294.64" y="142.24"/>
 <instance part="TP27" gate="G$1" x="294.64" y="139.7"/>
-<instance part="TP29" gate="G$1" x="294.64" y="134.62"/>
+<instance part="TP28" gate="G$1" x="294.64" y="134.62"/>
 <instance part="GND16" gate="1" x="284.48" y="132.08"/>
 <instance part="+3V3" gate="G$1" x="284.48" y="147.32" smashed="yes">
@@
 <attribute name="VALUE" x="70.104" y="196.342" size="1.778" layer="96"/>
 </instance>
-<instance part="TP30" gate="G$1" x="294.64" y="137.16"/>
+<instance part="TP29" gate="G$1" x="294.64" y="137.16"/>
 </instances>
 <busses>
@@
 </segment>
 <segment>
-<pinref part="TP29" gate="G$1" pin="1"/>
+<pinref part="TP28" gate="G$1" pin="1"/>
 <pinref part="GND16" gate="1" pin="GND"/>
 <wire x1="292.1" y1="134.62" x2="284.48" y2="134.62" width="0.1524" layer="91"/>
@@
 <wire x1="261.62" y1="215.9" x2="292.1" y2="215.9" width="0.1524" layer="91"/>
 <label x="269.24" y="215.9" size="1.778" layer="95"/>
-<pinref part="TP28" gate="G$1" pin="1"/>
+<pinref part="TP26" gate="G$1" pin="1"/>
 </segment>
 </net>
@@
 <wire x1="261.62" y1="213.36" x2="292.1" y2="213.36" width="0.1524" layer="91"/>
 <label x="269.24" y="213.36" size="1.778" layer="95"/>
-<pinref part="TP3" gate="G$1" pin="1"/>
+<pinref part="TP2" gate="G$1" pin="1"/>
 </segment>
 <segment>
@@
 <wire x1="261.62" y1="210.82" x2="292.1" y2="210.82" width="0.1524" layer="91"/>
 <label x="269.24" y="210.82" size="1.778" layer="95"/>
-<pinref part="TP1" gate="G$1" pin="1"/>
+<pinref part="TP3" gate="G$1" pin="1"/>
 </segment>
 <segment>
@@
 <pinref part="U3" gate="G$1" pin="CT16B1_MAT0/MOSI1/PIO0_21"/>
 <wire x1="261.62" y1="170.18" x2="292.1" y2="170.18" width="0.1524" layer="91"/>
-<pinref part="TP2" gate="G$1" pin="1"/>
+<pinref part="TP1" gate="G$1" pin="1"/>
 <label x="269.748" y="170.18" size="1.778" layer="95"/>
 </segment>
@@
 <wire x1="261.62" y1="220.98" x2="292.1" y2="220.98" width="0.1524" layer="91"/>
 <label x="269.24" y="220.98" size="1.778" layer="95"/>
-<pinref part="TP26" gate="G$1" pin="1"/>
+<pinref part="TP25" gate="G$1" pin="1"/>
 </segment>
 <segment>
@@
 </segment>
 <segment>
-<pinref part="TP24" gate="G$1" pin="1"/>
+<pinref part="TP30" gate="G$1" pin="1"/>
 <wire x1="292.1" y1="142.24" x2="289.56" y2="142.24" width="0.1524" layer="91"/>
 <wire x1="289.56" y1="142.24" x2="289.56" y2="144.78" width="0.1524" layer="91"/>
@@
 <wire x1="261.62" y1="200.66" x2="292.1" y2="200.66" width="0.1524" layer="91"/>
 <label x="269.24" y="200.66" size="1.778" layer="95"/>
-<pinref part="TP25" gate="G$1" pin="1"/>
+<pinref part="TP24" gate="G$1" pin="1"/>
 </segment>
 </net>
@@
 <net name="AUX-VIN" class="0">
 <segment>
-<pinref part="TP30" gate="G$1" pin="1"/>
+<pinref part="TP29" gate="G$1" pin="1"/>
 <wire x1="292.1" y1="137.16" x2="271.78" y2="137.16" width="0.1524" layer="91"/>
 <label x="271.78" y="137.16" size="1.778" layer="95"/>

Commit message: Ready for final auto routing.
Parts:
- TP1: device ezlpc-proto:PINHD-1X1 -> ezlpc-proto:PINHD-1X1SQUARE
Changed lines of the file:
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@@
 <part name="TP18" library="ezlpc-proto" deviceset="PINHD-1X1" device=""/>
 <part name="TP21" library="ezlpc-proto" deviceset="PINHD-1X1" device=""/>
-<part name="TP1" library="ezlpc-proto" deviceset="PINHD-1X1" device=""/>
+<part name="TP1" library="ezlpc-proto" deviceset="PINHD-1X1" device="SQUARE"/>
 <part name="TP6" library="ezlpc-proto" deviceset="PINHD-1X1" device=""/>
 <part name="TP13" library="ezlpc-proto" deviceset="PINHD-1X1" device=""/>
