File: mini-pro/eagle/arm-mini-pro.brd (EAGLE design)
At the start: 38.1 x 20.3 mm, 61 parts, among them J1 MICRO USB, J2 SWD HEADER, Q1 12Mhz, T1 MMBT3906, U1 PRTR5V0U2X, U2 MIC5225-3.3v, U3 LPC11U35FHI33/501, U4 BAS40-05

Commit message: Renamed eagle files from ezlpc-proto to arm-mini-pro. Yet to do the same for the firmware.
Parts:
- C1, C2, C5, C6: device ezlpc-proto:C0603K -> arm-mini-pro:C0603K
- C3, C4: device ezlpc-proto:C0402K -> arm-mini-pro:C0402K
- J1: device ezlpc-proto:USB-MICRO-ZX62RD-AB-5P8 -> arm-mini-pro:USB-MICRO-ZX62RD-AB-5P8
- J2: device ezlpc-proto:SWD-HEADER -> arm-mini-pro:SWD-HEADER
- LED1, LED2, LED3: device ezlpc-proto:CHIP-LED0603 -> arm-mini-pro:CHIP-LED0603
- Q1: device ezlpc-proto:CRYSTAL -> arm-mini-pro:CRYSTAL
- R1, R10, R11, R12, R2, R3, R4, R5, R6, R7, R8, R9: device ezlpc-proto:R0402 -> arm-mini-pro:R0402
- S1, S2: device ezlpc-proto:PUSH_BUTTON -> arm-mini-pro:PUSH_BUTTON
- T1: device ezlpc-proto:SOT23-BEC -> arm-mini-pro:SOT23-BEC
- TP1: device ezlpc-proto:1X01-SQUARE -> arm-mini-pro:1X01-SQUARE
- TP10, TP11, TP12, TP13, TP14, TP15, TP16, TP17, TP18, TP19, TP2, TP20, TP21, TP22, TP23, TP24, TP25, TP26, TP27, TP28, TP29, TP3, TP30, TP4, TP5, TP6, TP7, TP8, TP9: device ezlpc-proto:1X01 -> arm-mini-pro:1X01
- U1: device ezlpc-proto:SOT143B -> arm-mini-pro:SOT143B
- U2: device ezlpc-proto:SOT25 -> arm-mini-pro:SOT25
- U3: device ezlpc-proto:HVQFN33-5MM -> arm-mini-pro:HVQFN33-5MM
- U4: device ezlpc-proto:SOT23 -> arm-mini-pro:SOT23

Commit message: Performed final auto routing.
Routing:
- net PIO0_7-LED: track 0.00 -> 63.8 mm, vias 0 -> 8
- net +3V3: track 40.2 -> 83.7 mm, vias 2 -> 5
- net PIO0_9-SWDO: track 0.00 -> 41.0 mm, vias 0 -> 3
- net PIO0_10-SWDCLK: track 0.00 -> 40.4 mm, vias 0 -> 6
- net GND: track 65.8 -> 105.8 mm, vias 8 -> 13
- net PIO0_1-ISP_EN: track 0.00 -> 32.1 mm, vias 0 -> 1
- net PIO0_0-RESET: track 0.00 -> 28.9 mm, vias 0 -> 1
- net PIO0_6-CONNECT: track 0.00 -> 27.0 mm, vias 0 -> 1
- net PIO0_15-SWDIO: track 0.00 -> 23.7 mm, vias 0 -> 1
- net PIO0_21: track 0.00 -> 22.0 mm, vias 0 -> 1
- net PIO0_3-VBUS: track 0.00 -> 21.9 mm, vias 0 -> 2
- net PIO0_18: track 0.00 -> 20.2 mm
- net PIO0_5: track 0.00 -> 17.3 mm, vias 0 -> 2
- net PIO0_17: track 0.00 -> 14.8 mm
- net PIO0_8: track 0.00 -> 13.9 mm
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- added copper zone on layer 16, net GND
