File: mini-pro/eagle/arm-mini-pro.sch (EAGLE design)
At the start: 61 parts, among them J1 MICRO USB, J2 SWD HEADER, Q1 12Mhz, T1 MMBT3906, U1 PRTR5V0U2X, U2 MIC5225-3.3v, U3 LPC11U35FHI33/501, U4 BAS40-05

Commit message: Renamed eagle files from ezlpc-proto to arm-mini-pro. Yet to do the same for the firmware.
Parts:
- C1, C2, C5, C6: device ezlpc-proto:CAPACITORC0603K -> arm-mini-pro:CAPACITORC0603K
- C3, C4: device ezlpc-proto:C-USC0402K -> arm-mini-pro:C-USC0402K
- J1: device ezlpc-proto:USB -> arm-mini-pro:USB
- J2: device ezlpc-proto:SWD-HEADER -> arm-mini-pro:SWD-HEADER
- LED1, LED2, LED3: device ezlpc-proto:LEDCHIP-LED0603 -> arm-mini-pro:LEDCHIP-LED0603
- Q1: device ezlpc-proto:CRYSTALCTS406 -> arm-mini-pro:CRYSTALCTS406
- R1, R10, R11, R12, R2, R3, R4, R5, R6, R7, R8, R9: device ezlpc-proto:R-US_R0402 -> arm-mini-pro:R-US_R0402
- S1, S2: device ezlpc-proto:PUSH_BUTTON -> arm-mini-pro:PUSH_BUTTON
- T1: device ezlpc-proto:BC857B-PNP-SOT23-BEC -> arm-mini-pro:BC857B-PNP-SOT23-BEC
- TP1: device ezlpc-proto:PINHD-1X1SQUARE -> arm-mini-pro:PINHD-1X1SQUARE
- TP10, TP11, TP12, TP13, TP14, TP15, TP16, TP17, TP18, TP19, TP2, TP20, TP21, TP22, TP23, TP24, TP25, TP26, TP27, TP28, TP29, TP3, TP30, TP4, TP5, TP6, TP7, TP8, TP9: device ezlpc-proto:PINHD-1X1 -> arm-mini-pro:PINHD-1X1
- U1: device ezlpc-proto:PRTR5V0U2X -> arm-mini-pro:PRTR5V0U2X
- U2: device ezlpc-proto:TC1015 -> arm-mini-pro:TC1015
- U3: device ezlpc-proto:LPC11U35FHN33/501 -> arm-mini-pro:LPC11U35FHN33/501
- U4: device ezlpc-proto:BAS40-05 -> arm-mini-pro:BAS40-05

Commit message: Added pdf files.
Other:
- note added: "1"
- note removed: "D"
- moved on the sheet: C1, C2, J2, R8, R9, U2, U4
