File: pro-mini/eagle/arm-pro-mini.sch (EAGLE design)
At the start: 61 parts, among them J1 MICRO USB, J2 SWD HEADER, Q1 12Mhz, T1 MMBT3906, U1 PRTR5V0U2X, U2 MIC5225-3.3v, U3 LPC11U35FHI33/501, U4 BAS40-05

Commit message: Moved the SWD header slightly up to increase the clearance from the buttons.
Other:
- note added: "1B"
- note removed: "1A"
Changed lines of the file:
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@@
 <wire x1="0" y1="0" x2="0" y2="259.08" width="0.1524" layer="94"/>
 <text x="226.06" y="137.16" size="2.54" layer="97">MCU</text>
-<text x="331.978" y="7.112" size="2.54" layer="97">1A</text>
+<text x="331.978" y="7.112" size="2.54" layer="97">1B</text>
 <text x="73.914" y="48.26" size="2.54" layer="97">3.3V REGULATOR</text>
 <text x="66.04" y="114.3" size="2.54" layer="97">USB</text>
