File: pro-mini/eagle/arm-pro-mini.sch (EAGLE design)
At the start: 61 parts, among them J1 MICRO USB, J2 SWD HEADER, Q1 12Mhz, T1 MMBT3906, U1 PRTR5V0U2X, U2 MIC5225-3.3v, U3 LPC11U35FHI33/501, U4 BAS40-05

Commit message: Updatd license note.
Other:
- note added: "OSH. Share alike and attributions are optional. Commercial use ok."
Changed lines of the file:
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@@
 <wire x1="119.38" y1="53.34" x2="119.38" y2="86.36" width="0.1524" layer="97" style="shortdash"/>
 <text x="87.63" y="56.388" size="1.778" layer="94">Optional C</text>
+<text x="10.16" y="7.62" size="2.54" layer="97" font="vector">OSH. Share alike and attributions are optional. Commercial use ok.</text>
 </plain>
 <instances>

Commit message: Changed R4, R11 from 1.5K to 10K. R4 to reduce max current via MCU protection diodes and R11 to make the red LED less bright.
Parts:
- R11, R4: value 1K5 -> 10K
Changed lines of the file:
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@@
 <part name="S2" library="arm-pro-mini" deviceset="PUSH_BUTTON" device=""/>
 <part name="GND14" library="arm-pro-mini" deviceset="GND" device=""/>
-<part name="R4" library="arm-pro-mini" deviceset="R-US_" device="R0402" value="1K5"/>
+<part name="R4" library="arm-pro-mini" deviceset="R-US_" device="R0402" value="10K"/>
 <part name="+3V9" library="arm-pro-mini" deviceset="+3V3" device=""/>
 <part name="R2" library="arm-pro-mini" deviceset="R-US_" device="R0402" value="10K"/>
@@
 <part name="R12" library="arm-pro-mini" deviceset="R-US_" device="R0402" value="10K"/>
 <part name="GND5" library="arm-pro-mini" deviceset="GND" device=""/>
-<part name="R11" library="arm-pro-mini" deviceset="R-US_" device="R0402" value="1K5"/>
+<part name="R11" library="arm-pro-mini" deviceset="R-US_" device="R0402" value="10K"/>
 <part name="R7" library="arm-pro-mini" deviceset="R-US_" device="R0402" value="1K5"/>
 <part name="LED2" library="arm-pro-mini" deviceset="LED" device="CHIP-LED0603" value="Red"/>
