File: pro-tiny/eagle/arm-pro-tiny.brd (EAGLE design)
At the start: 20.3 x 17.8 mm, 26 parts, among them J1 USB, Q1 12Mhz, U1 MIC5225-3.3v, U2 LPC11U35FHI33/501

Commit message: Layout completed.
Parts:
- moved J1 0.43 mm to (-0.53, 8.89)
Routing:
- net PIO0_9: track 8.73 -> 8.07 mm
- net USB_DM: track 5.82 -> 5.25 mm
Other:
- board text added: "1"
- board text added: "12"
- board text added: "6"
- board text added: "7"
- board text added: "TP1"
- board text added: "TP10"
- board text added: "TP11"
- board text added: "TP12"
- board text added: "TP2"
- board text added: "TP3"
- board text added: "TP4"
- board text added: "TP5"
- board text added: "TP6"
- board text added: "TP7"
- board text added: "TP8"
- board text added: "TP9"

Commit message: Updatd license note.
Other:
- board text added: "OSH. Share alike and attributions are optional. Commercial use ok."
Changed lines of the file:
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@@
 <setting verticaltext="up"/>
 </settings>
-<grid distance="10" unitdist="mil" unit="mil" style="lines" multiple="1" display="no" altdistance="0.001" altunitdist="inch" altunit="inch"/>
+<grid distance="25" unitdist="mil" unit="mil" style="lines" multiple="1" display="no" altdistance="0.001" altunitdist="inch" altunit="inch"/>
 <layers>
 <layer number="1" name="Top" color="4" fill="1" visible="yes" active="yes"/>
@@
 <text x="19.6596" y="15.4432" size="0.8128" layer="25" font="vector" ratio="10" rot="R180">7</text>
 <text x="2.1336" y="15.4432" size="0.8128" layer="25" font="vector" ratio="10" rot="R180">12</text>
-<text x="0.762" y="-0.254" size="0.8128" layer="48" font="vector" ratio="10" rot="R270">TP1</text>
-<text x="3.302" y="-0.254" size="0.8128" layer="48" font="vector" ratio="10" rot="R270">TP2</text>
-<text x="5.842" y="-0.254" size="0.8128" layer="48" font="vector" ratio="10" rot="R270">TP3</text>
-<text x="13.462" y="-0.254" size="0.8128" layer="48" font="vector" ratio="10" rot="R270">TP4</text>
-<text x="16.002" y="-0.254" size="0.8128" layer="48" font="vector" ratio="10" rot="R270">TP5</text>
-<text x="18.542" y="-0.254" size="0.8128" layer="48" font="vector" ratio="10" rot="R270">TP6</text>
-<text x="1.524" y="18.034" size="0.8128" layer="48" font="vector" ratio="10" rot="R90">TP12</text>
-<text x="4.064" y="18.034" size="0.8128" layer="48" font="vector" ratio="10" rot="R90">TP11</text>
-<text x="6.604" y="18.034" size="0.8128" layer="48" font="vector" ratio="10" rot="R90">TP10</text>
-<text x="14.224" y="18.034" size="0.8128" layer="48" font="vector" ratio="10" rot="R90">TP9</text>
-<text x="16.764" y="18.034" size="0.8128" layer="48" font="vector" ratio="10" rot="R90">TP8</text>
-<text x="19.304" y="18.034" size="0.8128" layer="48" font="vector" ratio="10" rot="R90">TP7</text>
+<text x="0.762" y="-0.889" size="0.8128" layer="48" font="vector" ratio="10" rot="R270">TP1</text>
+<text x="3.302" y="-0.889" size="0.8128" layer="48" font="vector" ratio="10" rot="R270">TP2</text>
+<text x="5.842" y="-0.889" size="0.8128" layer="48" font="vector" ratio="10" rot="R270">TP3</text>
+<text x="13.462" y="-0.889" size="0.8128" layer="48" font="vector" ratio="10" rot="R270">TP4</text>
+<text x="16.002" y="-0.889" size="0.8128" layer="48" font="vector" ratio="10" rot="R270">TP5</text>
+<text x="18.542" y="-0.889" size="0.8128" layer="48" font="vector" ratio="10" rot="R270">TP6</text>
+<text x="1.524" y="18.669" size="0.8128" layer="48" font="vector" ratio="10" rot="R90">TP12</text>
+<text x="4.064" y="18.669" size="0.8128" layer="48" font="vector" ratio="10" rot="R90">TP11</text>
+<text x="6.604" y="18.669" size="0.8128" layer="48" font="vector" ratio="10" rot="R90">TP10</text>
+<text x="14.224" y="18.669" size="0.8128" layer="48" font="vector" ratio="10" rot="R90">TP9</text>
+<text x="16.764" y="18.669" size="0.8128" layer="48" font="vector" ratio="10" rot="R90">TP8</text>
+<text x="19.304" y="18.669" size="0.8128" layer="48" font="vector" ratio="10" rot="R90">TP7</text>
+<text x="-0.09150625" y="-7.971884375" size="0.8128" layer="48" font="vector" ratio="10">OSH. Share alike and attributions
+are optional. Commercial use ok.</text>
 </plain>
 <attributes>
@@
 </board>
 </drawing>
+<compatibility>
+<note version="6.3" minversion="6.2.2" severity="warning">
+Since Version 6.2.2 text objects can contain more than one line,
+which will not be processed correctly with this version.
+</note>
+</compatibility>
 </eagle>
