File: pro-mini/eagle_temp/arm-pro-mini.sch (EAGLE design)
At the start: 55 parts, among them J1 USB, J2 SWD HEADER, Q1 12Mhz, T1 DTA114EET1G (2 X 10K), U1 MCP1754ST-3302E/CB, U2 NUF2042XV6T1G, U3 LPC11U35FHI33/501

Commit message: Updated arm-pro-mini (new/temp)
Parts:
- R1: value 1k5 -> 1K5
- R6: value 10K -> 1K5
Other:
- note added: "2D"
- note removed: "2C"
- moved on the sheet: C1, C2, U1
Changed lines of the file:
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@@
 <part name="+3V2" library="arm-pro-mini" deviceset="+3V3" device=""/>
 <part name="GND8" library="arm-pro-mini" deviceset="GND" device=""/>
-<part name="R1" library="arm-pro-mini" deviceset="R-US_" device="R0402" value="1k5"/>
+<part name="R1" library="arm-pro-mini" deviceset="R-US_" device="R0402" value="1K5"/>
 <part name="P+4" library="arm-pro-mini" deviceset="USB-5V" device=""/>
 <part name="+3V5" library="arm-pro-mini" deviceset="+3V3" device=""/>
@@
 <part name="R2" library="arm-pro-mini" deviceset="R-US_" device="R0402" value="10K"/>
 <part name="+3V9" library="arm-pro-mini" deviceset="+3V3" device=""/>
-<part name="R6" library="arm-pro-mini" deviceset="R-US_" device="R0402" value="10K"/>
+<part name="R6" library="arm-pro-mini" deviceset="R-US_" device="R0402" value="1K5"/>
 <part name="GND5" library="arm-pro-mini" deviceset="GND" device=""/>
 <part name="R7" library="arm-pro-mini" deviceset="R-US_" device="R0402" value="10K"/>
@@
 <wire x1="0" y1="0" x2="0" y2="259.08" width="0.1524" layer="94"/>
 <text x="233.68" y="144.78" size="2.54" layer="97">MCU</text>
-<text x="331.978" y="7.112" size="2.54" layer="97">2C</text>
-<text x="78.994" y="48.26" size="2.54" layer="97">3.3V REGULATOR</text>
+<text x="331.978" y="7.112" size="2.54" layer="97">2D</text>
+<text x="68.834" y="48.26" size="2.54" layer="97">3.3V REGULATOR</text>
 <text x="71.12" y="149.86" size="2.54" layer="97">USB</text>
 <text x="154.94" y="48.26" size="2.54" layer="97">SWD DEBUGGER PORT
@@
 <text x="248.412" y="72.898" size="1.778" layer="94">PWR</text>
 <text x="261.62" y="48.26" size="2.54" layer="97">USER INTERFACE</text>
-<text x="25.654" y="48.26" size="2.54" layer="97">POWER SELECTOR</text>
+<text x="20.574" y="48.26" size="2.54" layer="97">POWER SELECTOR</text>
 <text x="10.16" y="7.62" size="2.54" layer="97" font="vector">OSH. Share alike and attributions are optional. Commercial use ok.</text>
 <text x="71.12" y="149.86" size="2.54" layer="97">USB</text>
@@
 <attribute name="NAME" x="301.752" y="71.628" size="1.778" layer="95"/>
 </instance>
-<instance part="GND3" gate="1" x="93.98" y="66.04"/>
-<instance part="C2" gate="G$1" x="109.22" y="76.2" smashed="yes">
-<attribute name="NAME" x="110.998" y="77.343" size="1.778" layer="95"/>
-<attribute name="VALUE" x="110.49" y="71.755" size="1.778" layer="96"/>
-</instance>
-<instance part="GND18" gate="1" x="109.22" y="66.04"/>
-<instance part="C1" gate="G$1" x="78.74" y="76.2" smashed="yes">
-<attribute name="NAME" x="73.152" y="77.343" size="1.778" layer="95"/>
-<attribute name="VALUE" x="72.898" y="71.755" size="1.778" layer="96"/>
-</instance>
-<instance part="GND28" gate="1" x="78.74" y="66.04"/>
+<instance part="GND3" gate="1" x="81.28" y="66.04"/>
+<instance part="C2" gate="G$1" x="96.52" y="76.2" smashed="yes">
+<attribute name="NAME" x="98.298" y="77.343" size="1.778" layer="95"/>
+<attribute name="VALUE" x="97.79" y="71.755" size="1.778" layer="96"/>
+</instance>
+<instance part="GND18" gate="1" x="96.52" y="66.04"/>
+<instance part="C1" gate="G$1" x="66.04" y="76.2" smashed="yes">
+<attribute name="NAME" x="60.452" y="77.343" size="1.778" layer="95"/>
+<attribute name="VALUE" x="60.198" y="71.755" size="1.778" layer="96"/>
+</instance>
+<instance part="GND28" gate="1" x="66.04" y="66.04"/>
 <instance part="U3" gate="G$1" x="254" y="190.5" smashed="yes">
 <attribute name="NAME" x="214.122" y="153.5176" size="1.778" layer="95"/>
@@
 <attribute name="VALUE" x="43.18" y="193.04" size="1.778" layer="96"/>
 </instance>
-<instance part="+3V5" gate="G$1" x="127" y="83.82" rot="R270"/>
+<instance part="+3V5" gate="G$1" x="114.3" y="83.82" rot="R270"/>
 <instance part="J2" gate="A" x="160.02" y="83.82"/>
 <instance part="+3V6" gate="G$1" x="149.86" y="104.14"/>
@@
 <instance part="D1" gate="G$1" x="271.78" y="71.12"/>
 <instance part="D2" gate="G$1" x="254" y="71.12"/>
-<instance part="U1" gate="G$1" x="93.98" y="78.74" smashed="yes">
-<attribute name="NAME" x="88.9" y="93.98" size="1.778" layer="95"/>
-<attribute name="VALUE" x="88.9" y="88.9" size="1.778" layer="96"/>
+<instance part="U1" gate="G$1" x="81.28" y="78.74" smashed="yes">
+<attribute name="NAME" x="76.2" y="93.98" size="1.778" layer="95"/>
+<attribute name="VALUE" x="76.2" y="88.9" size="1.778" layer="96"/>
 </instance>
 <instance part="J1" gate="G$1" x="35.56" y="170.18"/>
@@
 </segment>
 <segment>
-<wire x1="93.98" y1="71.12" x2="93.98" y2="68.58" width="0.1524" layer="91"/>
+<wire x1="81.28" y1="71.12" x2="81.28" y2="68.58" width="0.1524" layer="91"/>
 <pinref part="GND3" gate="1" pin="GND"/>
 <pinref part="U1" gate="G$1" pin="GND"/>
@@
 <pinref part="C2" gate="G$1" pin="2"/>
 <pinref part="GND18" gate="1" pin="GND"/>
-<wire x1="109.22" y1="71.12" x2="109.22" y2="68.58" width="0.1524" layer="91"/>
+<wire x1="96.52" y1="71.12" x2="96.52" y2="68.58" width="0.1524" layer="91"/>
 </segment>
 <segment>
 <pinref part="GND28" gate="1" pin="GND"/>
 <pinref part="C1" gate="G$1" pin="2"/>
-<wire x1="78.74" y1="68.58" x2="78.74" y2="71.12" width="0.1524" layer="91"/>
+<wire x1="66.04" y1="68.58" x2="66.04" y2="71.12" width="0.1524" layer="91"/>
 </segment>
 <segment>
@@
 </segment>
 <segment>
-<wire x1="104.14" y1="83.82" x2="109.22" y2="83.82" width="0.1524" layer="91"/>
+<wire x1="91.44" y1="83.82" x2="96.52" y2="83.82" width="0.1524" layer="91"/>
 <pinref part="C2" gate="G$1" pin="1"/>
-<wire x1="109.22" y1="83.82" x2="124.46" y2="83.82" width="0.1524" layer="91"/>
-<wire x1="109.22" y1="78.74" x2="109.22" y2="83.82" width="0.1524" layer="91"/>
-<junction x="109.22" y="83.82"/>
+<wire x1="96.52" y1="83.82" x2="111.76" y2="83.82" width="0.1524" layer="91"/>
+<wire x1="96.52" y1="78.74" x2="96.52" y2="83.82" width="0.1524" layer="91"/>
+<junction x="96.52" y="83.82"/>
 <pinref part="+3V5" gate="G$1" pin="+3V3"/>
 <pinref part="U1" gate="G$1" pin="VOUT"/>
@@
 <net name="N$10" class="0">
 <segment>
-<wire x1="83.82" y1="83.82" x2="78.74" y2="83.82" width="0.1524" layer="91"/>
+<wire x1="71.12" y1="83.82" x2="66.04" y2="83.82" width="0.1524" layer="91"/>
 <pinref part="C1" gate="G$1" pin="1"/>
-<wire x1="78.74" y1="78.74" x2="78.74" y2="83.82" width="0.1524" layer="91"/>
+<wire x1="66.04" y1="78.74" x2="66.04" y2="83.82" width="0.1524" layer="91"/>
 <pinref part="D3" gate="G$1" pin="C"/>
-<junction x="78.74" y="83.82"/>
-<junction x="78.74" y="83.82"/>
-<wire x1="48.26" y1="83.82" x2="78.74" y2="83.82" width="0.1524" layer="91"/>
+<junction x="66.04" y="83.82"/>
+<junction x="66.04" y="83.82"/>
+<wire x1="48.26" y1="83.82" x2="66.04" y2="83.82" width="0.1524" layer="91"/>
 <pinref part="U1" gate="G$1" pin="VIN"/>
 </segment>
