File: phone-finder/eagle/phone-finder.sch (EAGLE design)
At the start: 45 parts, among them J1 MICRO USB, J2 PHONE-JACK, K1 RELAY, Q1 DTA114EET1G (2x10K), Q2 2N2222, Q3 2N2222, T1 TRANSFORMER, U1 AP2114H-3.3TRG1, U2 NUF2042XV6T1G, U3 LPC11U35FHI33/501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

Commit message: Cleaned up the BOM.
Parts:
- R6: value 3K3 -> 3K
Changed lines of the file:
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@@
 <part name="GND7" library="phone-finder" deviceset="GND" device=""/>
 <part name="GND14" library="phone-finder" deviceset="GND" device=""/>
-<part name="R6" library="phone-finder" deviceset="R" device="R0402" value="3K3"/>
+<part name="R6" library="phone-finder" deviceset="R" device="R0402" value="3K"/>
 <part name="GND27" library="phone-finder" deviceset="GND" device=""/>
 <part name="ANTENNA" library="phone-finder" deviceset="PINHD-1X1" device=""/>
