File: ir-control/eagle/ir-control.brd (EAGLE design)
At the start: 40 x 45 mm, 35 parts, among them J1 MICRO USB, J2 MICRO USB, J3 MICRO USB, J4 SJ1-3523NG, Q1 DTA114EET1G (2x10K), Q2 12Mhz, Q3 MMBT2222A, U1 NUF2042XV6T1G, U2 MCP1754ST-3302E/CB, U3 LPC11U35FHI33/501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

Commit message: Performed final auto routing.
Routing:
- net !ISP_EN: track 0.17 -> 60.9 mm, vias 0 -> 2
- net !RESET: track 0.00 -> 52.1 mm, vias 0 -> 4
- net LED: track 0.00 -> 43.6 mm, vias 0 -> 2
- net !TV_ON: track 0.00 -> 35.0 mm, vias 0 -> 2
- net +5V: track 29.8 -> 50.0 mm
- net !AV_ON: track 0.00 -> 15.3 mm, vias 0 -> 2
- net N$8: track 0.00 -> 14.7 mm
- net +3V3: track 64.3 -> 78.4 mm, vias 2 -> 4
- net IR: track 0.00 -> 11.1 mm, vias 0 -> 2
- net N$14: track 0.00 -> 6.92 mm
- net N$9: track 0.00 -> 6.06 mm
- net N$16: track 4.15 -> 8.97 mm
- net !USB_CONNECT: track 0.00 -> 3.87 mm
- net N$4: track 0.07 -> 1.89 mm
- added copper zone on layer 16, net GND
