File: ir-control/eagle/ir-control.brd (EAGLE design)
At the start: 40 x 45 mm, 35 parts, among them J1 MICRO USB, J2 MICRO USB, J3 MICRO USB, J4 SJ1-3523NG, Q1 DTA114EET1G (2x10K), Q2 12Mhz, Q3 MMBT2222A, U1 NUF2042XV6T1G, U2 MCP1754ST-3302E/CB, U3 LPC11U35FHI33/501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

Commit message: Minor tweaks, change IR resistor from 330R to 100R, reduce IR TX timeout.
Parts:
- R7: value 330 -> 100
Changed lines of the file:
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@@
 <attribute name="MF" value="" x="30" y="35" size="1.778" layer="27" rot="R180" display="off"/>
 </element>
-<element name="R7" library="ir-control" package="R0402" value="330" x="24.431" y="37.592" smashed="yes" rot="R180">
+<element name="R7" library="ir-control" package="R0402" value="100" x="24.431" y="37.592" smashed="yes" rot="R180">
 <attribute name="NAME" x="23.702" y="35.814" size="1.016" layer="25" font="vector" ratio="10"/>
 </element>
